File: Pedals/TrueBypass/bypass.sch (EAGLE design)
At the start: 7 parts

Commit message: Route board
Parts:
- removed S1: SWITCH-3PDT-PTH-STOMP, SparkFun-Switches:SWITCH-3PDT-PTH-STOMP
- added SW1: (no value), mb_3pdt:3PDT
Connections:
- net N$1: now also SW1A.P$2; no longer S1A.P
- net N$2: now also SW1B.P$2; no longer S1B.P
- net N$3: now also SW1A.P$1, SW1B.P$1; no longer S1A.O, S1B.O
- net N$4: now also SW1C.P$3; no longer S1C.S
- net N$5: now also SW1A.P$3; no longer S1A.S
- net N$6: now also SW1B.P$3; no longer S1B.S
- net N$7: now also SW1C.P$2; no longer S1C.P
Changed lines of the file:
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@@
 </classes>
 <parts>
-<part name="S1" library="SparkFun-Switches" library_urn="urn:adsk.eagle:library:535" deviceset="SWITCH-3PDT" device="-PTH-STOMP" package3d_urn="urn:adsk.eagle:package:40159/1"/>
 <part name="OUT_JACK" library="Custom-Parts" deviceset="CONN_02" device="POLAR" package3d_urn="urn:adsk.eagle:package:38040/1"/>
 <part name="IN_JACK" library="Custom-Parts" deviceset="CONN_02" device="POLAR" package3d_urn="urn:adsk.eagle:package:38040/1"/>
@@
 <part name="U$5" library="SparkFun-PowerSymbols" library_urn="urn:adsk.eagle:library:530" deviceset="AGND" device=""/>
 <part name="R1" library="SparkFun-Resistors" library_urn="urn:adsk.eagle:library:532" deviceset="330OHM" device="-HORIZ-1/10W-5%" package3d_urn="urn:adsk.eagle:package:39658/1" value="330"/>
+<part name="SW1" library="mb_3pdt" deviceset="3PDT" device=""/>
 </parts>
 <sheets>
@@
 </plain>
 <instances>
-<instance part="S1" gate="A" x="25.4" y="86.36" smashed="yes">
-<attribute name="NAME" x="24.13" y="89.662" size="1.778" layer="95" font="vector" align="bottom-center"/>
-</instance>
-<instance part="S1" gate="B" x="25.4" y="63.5" smashed="yes">
-<attribute name="NAME" x="24.13" y="66.802" size="1.778" layer="95" font="vector" align="bottom-center"/>
-</instance>
-<instance part="S1" gate="C" x="25.4" y="38.1" smashed="yes">
-<attribute name="NAME" x="24.13" y="41.402" size="1.778" layer="95" font="vector" align="bottom-center"/>
-</instance>
 <instance part="OUT_JACK" gate="G$1" x="7.62" y="60.96" smashed="yes">
 <attribute name="VALUE" x="5.08" y="56.134" size="1.778" layer="96" font="vector"/>
@@
 <attribute name="NAME" x="43.18" y="37.084" size="1.778" layer="95" font="vector" align="bottom-center"/>
 <attribute name="VALUE" x="43.18" y="34.036" size="1.778" layer="96" font="vector" align="top-center"/>
+</instance>
+<instance part="SW1" gate="A" x="22.86" y="86.36" smashed="yes">
+<attribute name="NAME" x="17.145" y="88.9" size="1.4224" layer="95"/>
+</instance>
+<instance part="SW1" gate="B" x="22.86" y="63.5" smashed="yes">
+<attribute name="NAME" x="17.145" y="66.04" size="1.4224" layer="95"/>
+</instance>
+<instance part="SW1" gate="C" x="22.86" y="38.1" smashed="yes">
+<attribute name="NAME" x="17.145" y="40.64" size="1.4224" layer="95"/>
 </instance>
 </instances>
@@
 <segment>
 <pinref part="IN_JACK" gate="G$1" pin="2"/>
-<pinref part="S1" gate="A" pin="P"/>
 <wire x1="15.24" y1="86.36" x2="20.32" y2="86.36" width="0.1524" layer="91"/>
+<pinref part="SW1" gate="A" pin="P$2"/>
 </segment>
 </net>
@@
 <segment>
 <pinref part="OUT_JACK" gate="G$1" pin="2"/>
-<pinref part="S1" gate="B" pin="P"/>
 <wire x1="15.24" y1="63.5" x2="20.32" y2="63.5" width="0.1524" layer="91"/>
+<pinref part="SW1" gate="B" pin="P$2"/>
 </segment>
 </net>
 <net name="N$3" class="0">
 <segment>
-<pinref part="S1" gate="A" pin="O"/>
 <wire x1="27.94" y1="88.9" x2="33.02" y2="88.9" width="0.1524" layer="91"/>
 <wire x1="33.02" y1="88.9" x2="33.02" y2="66.04" width="0.1524" layer="91"/>
-<pinref part="S1" gate="B" pin="O"/>
 <wire x1="33.02" y1="66.04" x2="27.94" y2="66.04" width="0.1524" layer="91"/>
+<pinref part="SW1" gate="A" pin="P$1"/>
+<pinref part="SW1" gate="B" pin="P$1"/>
 </segment>
 </net>
 <net name="N$5" class="0">
 <segment>
-<pinref part="S1" gate="A" pin="S"/>
 <wire x1="27.94" y1="83.82" x2="27.94" y2="73.66" width="0.1524" layer="91"/>
 <pinref part="PCB" gate="G$1" pin="4"/>
 <wire x1="27.94" y1="73.66" x2="50.8" y2="73.66" width="0.1524" layer="91"/>
+<pinref part="SW1" gate="A" pin="P$3"/>
 </segment>
 </net>
 <net name="N$6" class="0">
 <segment>
-<pinref part="S1" gate="B" pin="S"/>
 <wire x1="27.94" y1="60.96" x2="38.1" y2="60.96" width="0.1524" layer="91"/>
 <wire x1="38.1" y1="60.96" x2="38.1" y2="76.2" width="0.1524" layer="91"/>
 <pinref part="PCB" gate="G$1" pin="3"/>
 <wire x1="38.1" y1="76.2" x2="50.8" y2="76.2" width="0.1524" layer="91"/>
+<pinref part="SW1" gate="B" pin="P$3"/>
 </segment>
 </net>
@@
 <segment>
 <pinref part="POWER" gate="G$1" pin="2"/>
-<pinref part="S1" gate="C" pin="P"/>
 <wire x1="15.24" y1="38.1" x2="20.32" y2="38.1" width="0.1524" layer="91"/>
+<pinref part="SW1" gate="C" pin="P$2"/>
 </segment>
 </net>
 <net name="N$4" class="0">
 <segment>
-<pinref part="S1" gate="C" pin="S"/>
 <wire x1="27.94" y1="35.56" x2="35.56" y2="35.56" width="0.1524" layer="91"/>
 <wire x1="35.56" y1="35.56" x2="35.56" y2="78.74" width="0.1524" layer="91"/>
@@
 <wire x1="38.1" y1="35.56" x2="35.56" y2="35.56" width="0.1524" layer="91"/>
 <junction x="35.56" y="35.56"/>
+<pinref part="SW1" gate="C" pin="P$3"/>
 </segment>
 </net>
