File: Pedals/Terrarium KiCad/Terrarium.kicad_pcb (KiCad board)
At the start: 2 copper layers, 59.4 x 73 mm, 46 parts, among them IC1 TL072CP, IC2 LM78L05, SW5 3PDTTOGGLE

Commit message: Update the board to Rev B
Other:
- board text added: "Terrarium Clone REV: B"
- board text removed: "Terrarium Clone REV: A"
Changed lines of the file:
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@@
 		(layer "Edge.Cuts")
 	)
-	(gr_text "Terrarium Clone\nREV: A"
+	(gr_text "Terrarium Clone\nREV: B"
 		(at 123.1391 134.1451 0)
 		(layer "F.SilkS")
