File: Pedals/Terrarium KiCad/Terrarium.kicad_sch (KiCad schematic)
At the start: 46 parts, among them IC1 TL072CP, IC2 LM78L05, SW1 SPDT.1, SW2 SPDT.1, SW3 SPDT.1, SW4 SPDT.1, SW5 3PDTTOGGLE

Commit message: Update board with new components
Parts:
- removed C1: 100p, Terrarium-import-fps:5MM, symbol Terrarium-eagle-import:CAP.2
- removed C100: 100u, Terrarium-import-fps:050_2.5MM.2, symbol Terrarium-eagle-import:5.0_MM.4
- removed C2, C3, C6: 1u, Terrarium-import-fps:.33UF+, symbol Terrarium-eagle-import:CAP.5
- removed C4, C5, C8, C9: 100n, Terrarium-import-fps:5MM, symbol Terrarium-eagle-import:CAP.2
- removed C7: 1n, Terrarium-import-fps:5MM, symbol Terrarium-eagle-import:CAP.2
- removed D100: 1N5817, Terrarium-import-fps:DO41-3, symbol Terrarium-eagle-import:DO41.3
- removed FS1, FS2: SPST, Terrarium-import-fps:SPST, symbol Terrarium-eagle-import:SPST
- removed GND0, IN0, IN_GND0, OUT0, OUT_GND0, PWR0: PADRD, Terrarium-import-fps:UNLABELED, symbol Terrarium-eagle-import:PADRD
- removed IC1: TL072CP, Terrarium-import-fps:DIP794W53P254L959H508Q8N, symbol Terrarium-eagle-import:TL072CP
- removed IC2: LM78L05, Terrarium-import-fps:TO92-, symbol Terrarium-eagle-import:LM78L05
- removed LED1, LED2, LED3: LED.3, Terrarium-import-fps:3MM_2, symbol Terrarium-eagle-import:LED.3
- removed POT1, POT2, POT3, POT4, POT5, POT6: B10K, Terrarium-import-fps:16MM_PADS.2, symbol Terrarium-eagle-import:16MM.5
- removed R1, R2, R3, R9: 1M, Terrarium-import-fps:7.5MM.2, symbol Terrarium-eagle-import:R.3B
- removed R10: 4.7K, Terrarium-import-fps:7.5MM.2, symbol Terrarium-eagle-import:R.3B
- removed R4: 100R, Terrarium-import-fps:7.5MM.2, symbol Terrarium-eagle-import:R.3B
- removed R5, R7, R8: 1K, Terrarium-import-fps:7.5MM.2, symbol Terrarium-eagle-import:R.3B
- removed R6: 100K, Terrarium-import-fps:7.5MM.2, symbol Terrarium-eagle-import:R.3B
- removed SW1, SW2, SW3, SW4: SPDT.1, Terrarium-import-fps:SPDT_SOLDER_LUG, symbol Terrarium-eagle-import:SPDT.1
- removed SW5: 3PDTTOGGLE, Terrarium-import-fps:3PDT2, symbol Terrarium-eagle-import:3PDTTOGGLE
- added C1, C20, C4: 100uF 16V, Capacitor_THT:CP_Radial_D6.3mm_P2.50mm, symbol Device:C_Polarized
- added C10, C14, C15: 1uF, Capacitor_THT:C_Rect_L7.2mm_W4.5mm_P5.00mm_FKS2_FKP2_MKS2_MKP2, symbol Device:C
- added C11: 100pF, Capacitor_THT:C_Disc_D3.0mm_W1.6mm_P2.50mm, symbol Device:C
- added C12: 1nF, Capacitor_THT:C_Disc_D3.0mm_W1.6mm_P2.50mm, symbol Device:C
- added C13: 2.2nF, Capacitor_THT:C_Disc_D5.0mm_W2.5mm_P5.00mm, symbol Device:C
- added C16: 470uF 16V, Capacitor_THT:CP_Radial_D8.0mm_P3.50mm, symbol Device:C_Polarized
- added C17: 330nF, Capacitor_THT:C_Disc_D5.0mm_W2.5mm_P5.00mm, symbol Device:C
- added C18: 10uF 16V, Capacitor_THT:CP_Radial_D5.0mm_P2.00mm, symbol Device:C_Polarized
- added C19, C21, C8: 100nF, Capacitor_THT:C_Disc_D3.0mm_W1.6mm_P2.50mm, symbol Device:C
- added C2, C3: 100nF, Capacitor_THT:C_Disc_D5.0mm_W2.5mm_P5.00mm, symbol Device:C
- added C5: 1uF, Capacitor_THT:C_Disc_D3.0mm_W1.6mm_P2.50mm, symbol Device:C
- added C6: 10nF, Capacitor_THT:C_Disc_D3.0mm_W1.6mm_P2.50mm, symbol Device:C
- added C7: 4.7uF, Capacitor_THT:C_Disc_D3.0mm_W1.6mm_P2.50mm, symbol Device:C
- added C9: 47uF 16V, Capacitor_THT:CP_Radial_D5.0mm_P2.00mm, symbol Device:C_Polarized
- added D1: 1N5817, Diode_THT:D_DO-41_SOD81_P10.16mm_Horizontal, symbol Diode:1N5817
- added GND1: GND, Terrarium-import-fps:UNLABELED, symbol Terrarium-eagle-import:PADRD
- added H1, H2, H3, H4: M3, MountingHole:MountingHole_3.2mm_M3, symbol Mechanical:MountingHole
- added IN1: IN, Terrarium-import-fps:UNLABELED, symbol Terrarium-eagle-import:PADRD
- added INGND1: IN GND, Terrarium-import-fps:UNLABELED, symbol Terrarium-eagle-import:PADRD
- added J10: SPDT + encoder, Connector_PinHeader_2.54mm:PinHeader_1x07_P2.54mm_Vertical, symbol Connector_Generic:Conn_01x07
- added J11: Pots, Connector_PinHeader_2.54mm:PinHeader_1x06_P2.54mm_Vertical, symbol Connector_Generic:Conn_01x06
- added J12: Spare GPIO, Connector_PinHeader_2.54mm:PinHeader_1x06_P2.54mm_Vertical, symbol Connector_Generic:Conn_01x06
- added J7: OLED SPI, Connector_PinHeader_2.54mm:PinHeader_1x07_P2.54mm_Vertical, symbol Connector_Generic:Conn_01x07
- added J8: LEDs, Connector_PinHeader_2.54mm:PinHeader_1x07_P2.54mm_Vertical, symbol Connector_Generic:Conn_01x07
- added J9: FX switches + tap, Connector_PinHeader_2.54mm:PinHeader_1x08_P2.54mm_Vertical, symbol Connector_Generic:Conn_01x08
- added LED1: LED 3mm, LED_THT:LED_D3.0mm, symbol Device:LED
- added OUT1: OUT, Terrarium-import-fps:UNLABELED, symbol Terrarium-eagle-import:PADRD
- added OUTGND1: OUT GND, Terrarium-import-fps:UNLABELED, symbol Terrarium-eagle-import:PADRD
- added PWR1: 9V, Terrarium-import-fps:UNLABELED, symbol Terrarium-eagle-import:PADRD
- added R1, R11: 10R, Resistor_THT:R_Axial_DIN0207_L6.3mm_D2.5mm_P7.62mm_Horizontal, symbol Device:R
- added R10: 4.7k, Resistor_THT:R_Axial_DIN0207_L6.3mm_D2.5mm_P7.62mm_Horizontal, symbol Device:R
- added R14, R5, R7: 1M, Resistor_THT:R_Axial_DIN0207_L6.3mm_D2.5mm_P7.62mm_Horizontal, symbol Device:R
- added R2, R3, R9: 100k, Resistor_THT:R_Axial_DIN0207_L6.3mm_D2.5mm_P7.62mm_Horizontal, symbol Device:R
- added R21, R22, R23, R24, R25, R26: 2.2k, Resistor_THT:R_Axial_DIN0207_L6.3mm_D2.5mm_P7.62mm_Horizontal, symbol Device:R
- added R30, R31, R32, R33, R34: 47R, Resistor_THT:R_Axial_DIN0207_L6.3mm_D2.5mm_P2.54mm_Vertical, symbol Device:R
- added R35: 10k, Resistor_THT:R_Axial_DIN0207_L6.3mm_D2.5mm_P2.54mm_Vertical, symbol Device:R
- added R4: 1k, Resistor_THT:R_Axial_DIN0207_L6.3mm_D2.5mm_P7.62mm_Horizontal, symbol Device:R
- added R6: 3.3k, Resistor_THT:R_Axial_DIN0207_L6.3mm_D2.5mm_P7.62mm_Horizontal, symbol Device:R
- added R8: 100R, Resistor_THT:R_Axial_DIN0207_L6.3mm_D2.5mm_P7.62mm_Horizontal, symbol Device:R
- added RN1: 10k, Resistor_THT:R_Array_SIP9, symbol Device:R_Network08
- added RN2: 10k, Resistor_THT:R_Array_SIP5, symbol Device:R_Network04
- added SW1: 3PDT, Terrarium-import-fps:3PDT2, symbol Terrarium-eagle-import:3PDTTOGGLE
- added U1: LP2985-5.0, Package_TO_SOT_SMD:SOT-23-5, symbol Regulator_Linear:LP2985-5.0
- added U2: MCP6022, Package_DIP:DIP-8_W7.62mm, symbol Amplifier_Operational:MCP6002-xP
- added U3: 78L05, Package_TO_SOT_THT:TO-92_Inline, symbol Regulator_Linear:L78L05_TO92
- SEED1: value ES_DAISY_SEED -> Daisy Seed / Seed3; IPN Daisy Seed -> (none)
Connections:
- net BYPASS: now also SW1.A3 (3), SW1.B3 (3)
- net GND: now also C1.2, C11.2, C12.2, C13.2, C16.2, C17.2, C18.2, C19.2, C2.2, C20.2, C21.2, C3.2, C4.2, C5.2, C6.2, C7.2, C8.2, C9.2, GND1.P$1, INGND1.P$1, J10.7 (Pin_7), J11.6 (Pin_6), J12.6 (Pin_6), J7.1 (Pin_1), J8.1 (Pin_1), LED1.1 (K), OUTGND1.P$1, R14.2, R3.2, R35.2, R9.2, RN1.1 (common), RN2.1 (common), U1.2 (GND), U2.4 (V-), U3.2 (GND)
- net FXLED1: now reaches SEED1.26 (GPIO19(ADC4))
- net FXLED1: now also R21.1
- net FXLED6: now reaches SEED1.23 (GPIO16(ADC1))
- net FXLED6: now also R26.1
- net FXLED4: now reaches SEED1.27 (GPIO20(ADC5))
- net FXLED4: now also R24.1
- net FXLED5: now reaches SEED1.25 (GPIO18(ADC3))
- net FXLED5: now also R25.1
- net FX4: now reaches SEED1.1 (GPIO0(USB_HS_ID))
- net FX4: now also J9.5 (Pin_5), RN1.5 (R4)
- net OLED_RES: now reaches SEED1.12 (GPIO11(I2C1_SCL))
- net OLED_RES: now also R32.1
- net SPDT_A: now reaches SEED1.13 (GPIO12(I2C1_SDA))
- net SPDT_A: now also J10.2 (Pin_2), RN1.9 (R8)
- net SPDT_B: now reaches SEED1.14 (GPIO13(USART1_TX))
- net SPDT_B: now also J10.3 (Pin_3), RN2.2 (R1)
- net EXT_D14: now reaches SEED1.15 (GPIO14(USART1_RX))
- net EXT_D14: now also J12.3 (Pin_3)
- net FX1: now reaches SEED1.2 (GPIO1(SDMMC1_D3))
- net FX1: now also J9.2 (Pin_2), RN1.2 (R1)
- net FXLED3: now reaches SEED1.22 (GPIO15(ADC0))
- net FXLED3: now also R23.1
- net FXLED2: now reaches SEED1.24 (GPIO17(ADC2))
- net FXLED2: now also R22.1
- net POT1: now reaches SEED1.28 (GPIO21(ADC6))
- net POT1: now also J11.2 (Pin_2)
- net FX5: now reaches SEED1.3 (GPIO2(SDMMC1_D2))
- net FX5: now also J9.6 (Pin_6), RN1.6 (R5)
- net POT4: now reaches SEED1.31 (GPIO24(ADC9))
- net POT4: now also J11.5 (Pin_5)
- net ENC_A: now reaches SEED1.34 (GPIO27(SAI2_FS_B))
- net ENC_A: now also J10.4 (Pin_4), RN2.3 (R2)
- net ENC_SW: now reaches SEED1.35 (GPIO28(ADC11))
- net ENC_SW: now also J10.6 (Pin_6), RN2.5 (R4)
- net EXT_D29: now reaches SEED1.36 (GPIO29(USB_HS_D_-))
- net EXT_D29: now also J12.5 (Pin_5)
- net TAP: now reaches SEED1.37 (GPIO30(USB_HS_D+))
- net TAP: now also J9.8 (Pin_8), RN1.8 (R7)
- net FX2: now reaches SEED1.4 (GPIO3(SDMMC1_D1))
- net FX2: now also J9.3 (Pin_3), RN1.3 (R2)
- net FX6: now reaches SEED1.5 (GPIO4(SDMMC1_D0))
- net FX6: now also J9.7 (Pin_7), RN1.7 (R6)
- net FX3: now reaches SEED1.6 (GPIO5(SDMMC1_CMD))
- net FX3: now also J9.4 (Pin_4), RN1.4 (R3)
- net EXT_D6: now reaches SEED1.7 (GPIO6(SDMMC1_CK))
- net EXT_D6: now also J12.2 (Pin_2)
- net 3V3_A renamed +3V3_A
- net +3V3_A: now also J11.1 (Pin_1)
- net 3V3_D renamed +3V3_D
- net +3V3_D: now also J10.1 (Pin_1), J12.1 (Pin_1), J9.1 (Pin_1)
- net FS1 renamed EXT_D25
- net EXT_D25: now also J12.4 (Pin_4)
- net FS2 renamed ENC_B
- net ENC_B: now also J10.5 (Pin_5), RN2.4 (R3)
- net LED1 renamed POT2
- net POT2: now also J11.3 (Pin_3)
- net LED2 renamed POT3
- net POT3: now also J11.4 (Pin_4)
- net LEFT_IN renamed SEED_IN_L
- net SEED_IN_L: now also U2.1, U2.2 (-)
- net LEFT_OUT renamed SEED_OUT_L
- net SEED_OUT_L: now also R6.1
- net SW1 renamed OLED_MOSI
- net OLED_MOSI: now also R31.1
- net SW2 renamed OLED_DC
- net OLED_DC: now also R33.1
- net SW3 renamed OLED_SCK
- net OLED_SCK: now also R30.1
- net SW4 renamed OLED_CS
- net OLED_CS: now also R34.1
- net VCC renamed +9V
- net +9V: now also C1.1, C2.1, C3.1, D1.1 (K), R1.1, R11.1, SW1.C2 (2)
- new net +5V_A: C7.1, C8.1, R2.1, U1.5 (VOUT), U2.8 (V+)
- new net +5V_D: C18.1, C19.1, C20.1, C21.1, J7.2 (Pin_2), U3.1 (VO)
- new net +9V_A: C4.1, C5.1, R1.2, U1.1 (VIN), U1.3 (ON/~{OFF})
- new net +9V_D: C16.1, C17.1, R11.2, U3.3 (VI)
- new net 9V_IN: D1.2 (A), PWR1.P$1
- new net BYP_LED_A: LED1.2 (A), R10.2
- new net BYP_LED_R: R10.1, SW1.C1 (1)
- new net FXLED1_R: J8.2 (Pin_2), R21.2
- new net FXLED2_R: J8.3 (Pin_3), R22.2
- new net FXLED3_R: J8.4 (Pin_4), R23.2
- new net FXLED4_R: J8.5 (Pin_5), R24.2
- new net FXLED5_R: J8.6 (Pin_6), R25.2
- new net FXLED6_R: J8.7 (Pin_7), R26.2
- new net IN_AC: C10.2, R4.1
- new net IN_BUF: C12.1, R4.2, R5.2, U2.3 (+)
- new net IN_FX: C10.1, C11.1, R14.1, SW1.A1 (1)
- new net JACK_IN: IN1.P$1, SW1.A2 (2)
- new net JACK_OUT: OUT1.P$1, SW1.B2 (2)
- new net LDO_BP: C6.1, U1.4 (BP)
- new net OLED_CS_R: J7.7 (Pin_7), R34.2
- new net OLED_DC_R: J7.6 (Pin_6), R33.2
- new net OLED_MOSI_R: J7.4 (Pin_4), R31.2
- new net OLED_RES_R: J7.5 (Pin_5), R32.2, R35.1
- new net OLED_SCK_R: J7.3 (Pin_3), R30.2
- new net OUT_BUF: C14.2, R7.2, U2.5 (+)
- new net OUT_DRV: R8.1, U2.6 (-), U2.7
- new net OUT_FX: C15.2, R9.1, SW1.B1 (1)
- new net OUT_LPF: C13.1, C14.1, R6.2
- new net OUT_R: C15.1, R8.2
- new net VBIAS: C9.1, R2.2, R3.1, R5.1, R7.1
- no-connect marks 0 -> 3
Other:
- note added: "Analog supply +5V_A (op-amps, bias only)"
- note added: "DNP on Firmament"
- note added: "Daisy Pedal Breakout - DaisyMulti / Firmament pin map. Firmament: build with DEV_BOARD undefined; leave the OLED group (J7, R30-R35, C20, C21) unfitted."
- note added: "Daisy Seed (pin map = DaisyMulti / Firmament PedalConfig.h)"
- note added: "Digital supply +5V_D (display) - pre-filtered so its load pulses stay off +9V"
- note added: "Effect LEDs (off-board, ~0.6 mA each)"
- note added: "Filtered audio bias (2.5 V)"
- note added: "Input buffer"
- note added: "Mounting"
- note added: "OLED header (DNP on Firmament)"
- note added: "Output: 22 kHz RC filter + buffer"
- note added: "Pots"
- note added: "Power input + reverse protection"
- note added: "Seed rev7 out-of-band filter"
- note added: "Spare GPIO"
- note added: "Switch inputs: active-high to +3V3_D, 10k pulldowns"
- note added: "True bypass (3PDT) + indicator"
- note added: "anti-pop pulldown"
- note added: "at Seed VIN"
- note added: "at U2 pin 8"
- note added: "holds display in reset until firmware runs"
- company: (none) -> Saved By Grace Software
- title: (none) -> Daisy Pedal Breakout

Commit message: Final base board changes
Parts:
- removed LED1: LED 3mm, LED_THT:LED_D3.0mm, symbol Device:LED
- added J13: Bypass LED, Connector_PinHeader_2.54mm:PinHeader_1x02_P2.54mm_Vertical, symbol Connector_Generic:Conn_01x02
Connections:
- net BYPASS: now also SW1.A1 (1), SW1.B1 (1); no longer SW1.A3 (3), SW1.B3 (3)
- net BYP_LED_A: now also J13.2 (Pin_2)
- net BYP_LED_R: now also SW1.C3 (3); no longer SW1.C1 (1)
- net GND: now also J13.1 (Pin_1)
- net IN_FX: now also SW1.A3 (3); no longer SW1.A1 (1)
- net OUT_FX: now also SW1.B3 (3); no longer SW1.B1 (1)
Other:
- note added: "mounted on bottom side"
- note added: "panel LED: 1 = cathode, 2 = anode"
Changed lines of the file:
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@@
 			)
 		)
-		(property "Description" ""
+		(property "Description" "mounted on bottom side"
 			(at 220.98 219.71 0)
 			(effects
@@
 		)
 	)
-	(label "IN_FX"
+	(label "BYPASS"
 		(at 218.44 212.09 90)
 		(effects
@@
 		)
 	)
-	(label "BYPASS"
+	(label "IN_FX"
 		(at 223.52 212.09 90)
 		(effects
 			(font
 				(size 1.27 1.27)
+			)
+			(justify left bottom)
+		)
+	)
+	(text "mounted on bottom side"
+		(exclude_from_sim no)
+		(at 218.44 229.87 0)
+		(effects
+			(font
+				(size 1.0 1.0)
 			)
 			(justify left bottom)
@@
 		)
 	)
-	(label "OUT_FX"
+	(label "BYPASS"
 		(at 238.76 212.09 90)
 		(effects
@@
 		)
 	)
-	(label "BYPASS"
+	(label "OUT_FX"
 		(at 243.84 212.09 90)
 		(effects
@@
 		)
 	)
-	(wire
-		(pts
-			(xy 259.08 214.63)
-			(xy 259.08 212.09)
-		)
-		(stroke
-			(width 0)
-			(type default)
-		)
-	)
-	(label "BYP_LED_R"
-		(at 259.08 212.09 90)
-		(effects
-			(font
-				(size 1.27 1.27)
-			)
-			(justify left bottom)
-		)
+	(no_connect
+		(at 259.08 214.63)
 	)
 	(wire
@@
 		)
 	)
-	(no_connect
-		(at 264.16 214.63)
+	(wire
+		(pts
+			(xy 264.16 214.63)
+			(xy 264.16 212.09)
+		)
+		(stroke
+			(width 0)
+			(type default)
+		)
+	)
+	(label "BYP_LED_R"
+		(at 264.16 212.09 90)
+		(effects
+			(font
+				(size 1.27 1.27)
+			)
+			(justify left bottom)
+		)
 	)
 	(symbol
@@
 	)
 	(symbol
-		(lib_id "Device:LED")
+		(lib_id "Connector_Generic:Conn_01x02")
 		(at 294.64 219.71 0)
 		(unit 1)
@@
 		(in_pos_files yes)
 		(dnp no)
-		(property "Reference" "LED1"
+		(property "Reference" "J13"
 			(at 298.45 217.17000000000002 0)
 			(effects
@@
 			)
 		)
-		(property "Value" "LED 3mm"
+		(property "Value" "Bypass LED"
 			(at 298.45 219.71 0)
 			(effects
@@
 			)
 		)
-		(property "Footprint" "LED_THT:LED_D3.0mm"
+		(property "Footprint" "Connector_PinHeader_2.54mm:PinHeader_1x02_P2.54mm_Vertical"
 			(at 294.64 219.71 0)
 			(effects
@@
 			)
 		)
-		(property "Description" ""
+		(property "Description" "panel LED: 1 = cathode, 2 = anode"
 			(at 294.64 219.71 0)
 			(effects
@@
 			(project "Terrarium"
 				(path "/e570cf6c-9924-44c7-bfd5-3e09fe1ff0d1"
-					(reference "LED1")
+					(reference "J13")
 					(unit 1)
 				)
@@
 	(wire
 		(pts
-			(xy 290.83 219.71)
-			(xy 288.29 219.71)
+			(xy 289.56 219.71)
+			(xy 287.02 219.71)
 		)
 		(stroke
@@
 	)
 	(label "GND"
-		(at 288.29 219.71 180)
+		(at 287.02 219.71 180)
 		(effects
 			(font
@@
 	(wire
 		(pts
-			(xy 298.45 219.71)
-			(xy 300.99 219.71)
+			(xy 289.56 222.25)
+			(xy 287.02 222.25)
 		)
 		(stroke
@@
 	)
 	(label "BYP_LED_A"
-		(at 300.99 219.71 0)
-		(effects
-			(font
-				(size 1.27 1.27)
+		(at 287.02 222.25 180)
+		(effects
+			(font
+				(size 1.27 1.27)
+			)
+			(justify right bottom)
+		)
+	)
+	(text "panel LED: 1 = cathode, 2 = anode"
+		(exclude_from_sim no)
+		(at 292.09999999999997 229.87 0)
+		(effects
+			(font
+				(size 1.0 1.0)
 			)
 			(justify left bottom)
@@
 	(rectangle
 		(start 150 200)
-		(end 350 240.32)
-		(stroke
-			(width 0)
+		(end 350 250.32)
+		(stroke
+			(width 0)
